File: hardware/6502motherboard/6502motherboard.kicad_pcb (KiCad board)
At the start: 2 copper layers, 100 x 100 mm, 31 parts, among them J1 AUX 5VDC, J2 POWER 5V, J3 GND, J4 NO 7502, J5 IO_8, J6 CLK, SW1 POWER, SW2 SW_Push, T1 DS-1813, U1 LM7805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

Commit message: rev 1.9 complete
Parts:
- added C10: 0.1uF, Capacitor_THT:C_Disc_D3.0mm_W1.6mm_P2.50mm, F.Cu at (90.2, 113.4)
- added C9: 0.1uF, Capacitor_THT:C_Disc_D3.0mm_W1.6mm_P2.50mm, F.Cu at (90.1, 94.0)
- moved J1 62.8 mm to (175.3, 69.5)
- moved J2 39.4 mm to (174.5, 81.4)
- moved U1 36.2 mm to (180.2, 120.4), turned to 180 degrees
- moved C8 33.0 mm to (166.2, 124.9), turned to 180 degrees
- moved C6 27.4 mm to (175.2, 115.0), turned to 180 degrees
- moved C7 27.3 mm to (180.3, 115.0), turned to 0 degrees
- moved J4 14.2 mm to (180.2, 108.5), turned to -90 degrees
- moved SW1 7.51 mm to (175.9, 93.8)
Routing:
- net VCC: track 351.0 -> 386.9 mm
- net /AUX GND: track 23.4 -> 15.8 mm
- net VDC_IN: track 11.4 -> 15.4 mm
