File: hardware/6502motherboard/6502motherboard.kicad_sch (KiCad schematic)
At the start: 30 parts, among them J1 AUX 5VDC, J2 POWER 5V, J3 GND, J4 NO 7502, J5 IO_8, SW1 POWER, SW2 SW_Push, T1 DS-1813, U1 LM7805, U3 74HCT273

Commit message: rev 1.8 new pcb optimized power routing
Parts:
- added J6: CLK, Connector_JST:JST_PH_B3B-PH-K_1x03_P2.00mm_Vertical, symbol Connector:Conn_01x03_Pin
Connections:
- net CLK: now also J6.1 (Pin_1)
- net GND: now also J6.3 (Pin_3)
- net VCC: now also J6.2 (Pin_2)
Changed lines of the file:
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@@
     (title "6502 Motherboard")
     (date "2023-11-01")
-    (rev "1.7")
+    (rev "1.8")
     (company "Mariano Luna")
   )
@@
     (stroke (width 0) (type default))
   )
+  (wire (pts (xy 164.465 163.195) (xy 167.005 163.195))
+    (stroke (width 0) (type default))
+  )
   (bus (pts (xy 99.06 27.305) (xy 96.52 24.765))
     (stroke (width 0) (type default))
@@
     (stroke (width 0) (type default))
   )
+  (wire (pts (xy 165.1 168.275) (xy 167.005 168.275))
+    (stroke (width 0) (type default))
+  )
   (wire (pts (xy 240.03 36.195) (xy 240.03 23.495))
     (stroke (width 0) (type default))
@@
     (stroke (width 0) (type default))
   )
+  (wire (pts (xy 164.465 165.735) (xy 167.005 165.735))
+    (stroke (width 0) (type default))
+  )
   (bus (pts (xy 71.755 50.8) (xy 69.215 50.8))
     (stroke (width 0) (type default))
@@
     )
   )
+  (global_label "CLK" (shape input) (at 165.1 168.275 180) (fields_autoplaced)
+    (effects (font (size 1.27 1.27)) (justify right))
+    (property "Intersheetrefs" "${INTERSHEET_REFS}" (at 158.5467 168.275 0)
+      (effects (font (size 1.27 1.27)) (justify right) hide)
+    )
+  )
   (global_label "~{IO_07}" (shape input) (at 130.81 85.725 0) (fields_autoplaced)
     (effects (font (size 1.27 1.27)) (justify left))
@@
     )
   )
+  (symbol (lib_id "Connector:Conn_01x03_Pin") (at 172.085 165.735 180) (unit 1)
+    (in_bom yes) (on_board yes) (dnp no) (fields_autoplaced)
+    (property "Reference" "J6" (at 173.99 164.465 0)
+      (effects (font (size 1.27 1.27)) (justify right))
+    )
+    (property "Value" "CLK" (at 173.99 167.005 0)
+      (effects (font (size 1.27 1.27)) (justify right))
+    )
+    (property "Footprint" "Connector_JST:JST_PH_B3B-PH-K_1x03_P2.00mm_Vertical" (at 172.085 165.735 0)
+      (effects (font (size 1.27 1.27)) hide)
+    )
+    (property "Datasheet" "~" (at 172.085 165.735 0)
+      (effects (font (size 1.27 1.27)) hide)
+    )
+    (pin "1")
+    (pin "2")
+    (pin "3")
+    (instances
+      (project "6502motherboard"
+        (path "/79b045e9-6697-4ebd-8cd3-5e519b22df02"
+          (reference "J6") (unit 1)
+        )
+      )
+    )
+  )
   (symbol (lib_id "power:GND") (at 256.54 134.62 0) (unit 1)
     (in_bom yes) (on_board yes) (dnp no) (fields_autoplaced)
@@
     )
   )
+  (symbol (lib_id "power:VCC") (at 164.465 165.735 90) (unit 1)
+    (in_bom yes) (on_board yes) (dnp no) (fields_autoplaced)
+    (property "Reference" "#PWR035" (at 168.275 165.735 0)
+      (effects (font (size 1.27 1.27)) hide)
+    )
+    (property "Value" "VCC" (at 161.29 165.735 90)
+      (effects (font (size 1.27 1.27)) (justify left))
+    )
+    (property "Footprint" "" (at 164.465 165.735 0)
+      (effects (font (size 1.27 1.27)) hide)
+    )
+    (property "Datasheet" "" (at 164.465 165.735 0)
+      (effects (font (size 1.27 1.27)) hide)
+    )
+    (pin "1")
+    (instances
+      (project "6502motherboard"
+        (path "/79b045e9-6697-4ebd-8cd3-5e519b22df02"
+          (reference "#PWR035") (unit 1)
+        )
+      )
+      (project "simple6502"
+        (path "/c0007eb4-077e-4f77-aad9-8dd15548af06"
+          (reference "#PWR014") (unit 1)
+        )
+        (path "/c0007eb4-077e-4f77-aad9-8dd15548af06/710f29f6-117a-4dcb-a5e3-826b377de52e"
+          (reference "#PWR039") (unit 1)
+        )
+      )
+    )
+  )
   (symbol (lib_id "power:VCC") (at 35.56 123.19 0) (unit 1)
     (in_bom yes) (on_board yes) (dnp no) (fields_autoplaced)
@@
         )
       )
+    )
+  )
+  (symbol (lib_id "power:GND") (at 164.465 163.195 270) (unit 1)
+    (in_bom yes) (on_board yes) (dnp no) (fields_autoplaced)
+    (property "Reference" "#PWR036" (at 158.115 163.195 0)
+      (effects (font (size 1.27 1.27)) hide)
+    )
+    (property "Value" "GND" (at 161.29 163.195 90)
+      (effects (font (size 1.27 1.27)) (justify right))
+    )
+    (property "Footprint" "" (at 164.465 163.195 0)
+      (effects (font (size 1.27 1.27)) hide)
+    )
+    (property "Datasheet" "" (at 164.465 163.195 0)
+      (effects (font (size 1.27 1.27)) hide)
+    )
+    (pin "1")
+    (instances
+      (project "6502motherboard"
+        (path "/79b045e9-6697-4ebd-8cd3-5e519b22df02"
+          (reference "#PWR036") (unit 1)
+        )
+      )
+      (project "simple6502"
+        (path "/c0007eb4-077e-4f77-aad9-8dd15548af06"
+          (reference "#PWR020") (unit 1)
+        )
+        (path "/c0007eb4-077e-4f77-aad9-8dd15548af06/710f29f6-117a-4dcb-a5e3-826b377de52e"
+          (reference "#PWR040") (unit 1)
+        )
+      )

Commit message: rev 1.9 complete
Parts:
- added C10, C9: 0.1uF, Capacitor_THT:C_Disc_D3.0mm_W1.6mm_P2.50mm, symbol Device:C
Connections:
- net GND: now also C10.2, C9.2
- net VCC: now also C10.1, C9.1
Other:
- moved on the sheet: C1, C2, C3, C4, C5
