File: hardware/simple6502/simple6502.kicad_pcb (KiCad board)
At the start: 2 copper layers, 100 x 100 mm, 43 parts, among them J1 Expansion Port, J2 USB Power, J3 CLK SEL, J4 FTDI Serial, J5 GND, J6 RESET, J7 POWER 5V, J8 AUX 5VDC, J9 ~{VP}, SW1 RESET, SW2 POWER, T1 DS1813-10+, U1 W65C02SxP, U2 MC68B50, U3 RAM 62256, U4 ROM 28C256, U5 74HCT00, U6 74LS30, U7 74HC138, X1 ACO-1MHz

Commit message: simple6502 Rev:1.6 Final
Other:
- board text added: "CLK"
Changed lines of the file:
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@@
       (disableapertmacros false)
       (usegerberextensions false)
-      (usegerberattributes true)
-      (usegerberadvancedattributes true)
-      (creategerberjobfile true)
+      (usegerberattributes false)
+      (usegerberadvancedattributes false)
+      (creategerberjobfile false)
       (dashed_line_dash_ratio 12.000000)
       (dashed_line_gap_ratio 3.000000)
@@
       (plotinvisibletext false)
       (sketchpadsonfab false)
-      (subtractmaskfromsilk false)
+      (subtractmaskfromsilk true)
       (outputformat 1)
       (mirror false)
-      (drillshape 1)
+      (drillshape 0)
       (scaleselection 1)
-      (outputdirectory "")
+      (outputdirectory "CAM/")
     )
   )
@@
     (effects (font (size 0.8 0.8) (thickness 0.15) bold) (justify left bottom))
   )
+  (gr_text "CLK" (at 76.93 51.18) (layer "F.SilkS")
+    (effects (font (size 0.8 1) (thickness 0.15) bold) (justify left bottom))
+  )
   (gr_text "SW-G" (at 55.19 140.26) (layer "F.SilkS")
