File: hardware/IO_Card/IO_Card.kicad_sch (KiCad schematic)
At the start: 6 parts, among them J1 6502 Edge, J2 6502 Pinheader, U1 W65C22NxP

Commit message: Rev: 0.5 basic VIA wiring
Parts:
- added D2: 1N6263, Diode_THT:D_DO-35_SOD27_P7.62mm_Horizontal, symbol Diode:1N6263
- added J3: Port A, Connector_PinHeader_2.54mm:PinHeader_2x07_P2.54mm_Horizontal, symbol Connector_Generic:Conn_02x07_Odd_Even
- added J4: Port B, Connector_PinHeader_2.54mm:PinHeader_2x07_P2.54mm_Horizontal, symbol Connector_Generic:Conn_02x07_Odd_Even
- added J5: IO Select, Connector_PinHeader_2.54mm:PinHeader_2x04_P2.54mm_Vertical, symbol Connector_Generic:Conn_02x04_Odd_Even
Connections:
- net A0: now also U1.38 (RS0)
- net A1: now also U1.37 (RS1)
- net A2: now also U1.36 (RS2)
- net A3: now also U1.35 (RS3)
- net CLK: now also U1.25 (ϕ2)
- net D0: now also U1.33 (D0)
- net D1: now also U1.32 (D1)
- net D2: now also U1.31 (D2)
- net D3: now also U1.30 (D3)
- net D4: now also U1.29 (D4)
- net D5: now also U1.28 (D5)
- net D6: now also U1.27 (D6)
- net D7: now also U1.26 (D7)
- net GND: now also J3.13 (Pin_13), J3.2 (Pin_2), J4.13 (Pin_13), J4.2 (Pin_2)
- net R~{W}: now also U1.22 (R/~{W})
- net VCC: now also J3.1 (Pin_1), J3.14 (Pin_14), J4.1 (Pin_1), J4.14 (Pin_14)
- net ~{IO_03}: now also J5.4 (Pin_4)
- net ~{IO_04}: now also J5.6 (Pin_6)
- net ~{IO_05}: now also J5.8 (Pin_8)
- net ~{IO_SLOT}: now also J5.2 (Pin_2)
- net ~{IRQ}: now also D2.2 (A)
- net ~{RESET}: now also U1.34 (~{RES})
- net PB0: now reaches U1.10 (PB0)
- net PB1: now reaches U1.11 (PB1)
- net PB1: now also J4.4 (Pin_4)
- net PB2: now reaches U1.12 (PB2)
- net PB3: now reaches U1.13 (PB3)
- net PB3: now also J4.6 (Pin_6)
- net PB4: now reaches U1.14 (PB4)
- net PB5: now reaches U1.15 (PB5)
- net PB5: now also J4.8 (Pin_8)
- net PB6: now reaches U1.16 (PB6)
- net PB7: now reaches U1.17 (PB7)
- net PB7: now also J4.10 (Pin_10)
- net CB1: now reaches U1.18 (CB1)
- net CB2: now reaches U1.19 (CB2)
- net CB2: now also J4.12 (Pin_12)
- net PA0: now reaches U1.2 (PA0)
- net PA0: now also J3.3 (Pin_3), J4.3 (Pin_3)
- net ~{IRQ_V1}: now reaches U1.21 (~{IRQ})
- net ~{IRQ_V1}: now also D2.1 (K)
- net ~{CS_V1}: now reaches U1.23 (~{CS2})
- net ~{CS_V1}: now also J5.1 (Pin_1), J5.3 (Pin_3), J5.5 (Pin_5), J5.7 (Pin_7)
- net PA1: now reaches U1.3 (PA1)
- net PA1: now also J3.4 (Pin_4)
- net CA2: now reaches U1.39 (CA2)
- net CA2: now also J3.12 (Pin_12)
- net PA2: now reaches U1.4 (PA2)
- net PA2: now also J3.5 (Pin_5), J4.5 (Pin_5)
- net CA1: now reaches U1.40 (CA1)
- net CA1: now also J3.11 (Pin_11), J4.11 (Pin_11)
- net PA3: now reaches U1.5 (PA3)
- net PA3: now also J3.6 (Pin_6)
- net PA4: now reaches U1.6 (PA4)
- net PA4: now also J3.7 (Pin_7), J4.7 (Pin_7)
- net PA5: now reaches U1.7 (PA5)
- net PA5: now also J3.8 (Pin_8)
- net PA6: now reaches U1.8 (PA6)
- net PA6: now also J3.9 (Pin_9), J4.9 (Pin_9)
- net PA7: now reaches U1.9 (PA7)
- net PA7: now also J3.10 (Pin_10)
Other:
- title: Protoboard Card -> IO Card - simple6502
- moved on the sheet: U1

Commit message: Rev 0.6 2 VIAs ready to route
Parts:
- added D3: 1N6263, Diode_THT:D_DO-35_SOD27_P7.62mm_Horizontal, symbol Diode:1N6263
- added J6: IO VIA2, Connector_PinHeader_2.54mm:PinHeader_2x04_P2.54mm_Vertical, symbol Connector_Generic:Conn_02x04_Odd_Even
- added J7: Port A, Connector_PinHeader_2.54mm:PinHeader_2x07_P2.54mm_Horizontal, symbol Connector_Generic:Conn_02x07_Odd_Even
- added J8: Port B, Connector_PinHeader_2.54mm:PinHeader_2x07_P2.54mm_Horizontal, symbol Connector_Generic:Conn_02x07_Odd_Even
- added R2, R3: 4K7, Resistor_THT:R_Axial_DIN0207_L6.3mm_D2.5mm_P10.16mm_Horizontal, symbol Device:R
- added U2: W65C22NxP, Package_DIP:DIP-40_W15.24mm, symbol PCM_65xx-library:W65C22NxP
- J5: value IO Select -> IO VIA1
Connections:
- net A0: now also U2.38 (RS0)
- net A1: now also U2.37 (RS1)
- net A2: now also U2.36 (RS2)
- net A3: now also U2.35 (RS3)
- net CLK: now also U2.25 (ϕ2)
- net D0: now also U2.33 (D0)
- net D1: now also U2.32 (D1)
- net D2: now also U2.31 (D2)
- net D3: now also U2.30 (D3)
- net D4: now also U2.29 (D4)
- net D5: now also U2.28 (D5)
- net D6: now also U2.27 (D6)
- net D7: now also U2.26 (D7)
- net GND: now also J7.13 (Pin_13), J7.2 (Pin_2), J8.13 (Pin_13), J8.2 (Pin_2), U2.1 (VSS)
- net PA0: no longer J4.3 (Pin_3)
- net PA2: no longer J4.5 (Pin_5)
- net PA4: no longer J4.7 (Pin_7)
- net PA6: no longer J4.9 (Pin_9)
- net PB0: now also J4.3 (Pin_3)
- net PB2: now also J4.5 (Pin_5)
- net PB4: now also J4.7 (Pin_7)
- net PB6: now also J4.9 (Pin_9)
- net R~{W}: now also U2.22 (R/~{W})
- net VCC: now also J7.1 (Pin_1), J7.14 (Pin_14), J8.1 (Pin_1), J8.14 (Pin_14), R2.2, R3.2, U2.20 (VCC)
- net ~{IO_04}: now also J6.4 (Pin_4); no longer J5.6 (Pin_6)
- net ~{IO_05}: now also J5.6 (Pin_6); no longer J5.8 (Pin_8)
- net ~{IO_06}: now also J6.6 (Pin_6)
- net ~{IO_07}: now also J5.8 (Pin_8)
- net ~{IO_CS}: now also J6.8 (Pin_8)
- net ~{IO_SLOT}: now also J6.2 (Pin_2)
- net ~{IRQ}: now also D3.2 (A)
- net ~{RESET}: now also U2.34 (~{RES})
- net at U1.24 (CS1): now also R3.1
- new net: R2.1, U2.24 (CS1)
- new net 2CA1: J7.11 (Pin_11), U2.40 (CA1)
- new net 2CA2: J7.12 (Pin_12), U2.39 (CA2)
- new net 2CB1: J8.11 (Pin_11), U2.18 (CB1)
- new net 2CB2: J8.12 (Pin_12), U2.19 (CB2)
- new net 2PA0: J7.3 (Pin_3), U2.2 (PA0)
- new net 2PA1: J7.4 (Pin_4), U2.3 (PA1)
- new net 2PA2: J7.5 (Pin_5), U2.4 (PA2)
- new net 2PA3: J7.6 (Pin_6), U2.5 (PA3)
- new net 2PA4: J7.7 (Pin_7), U2.6 (PA4)
- new net 2PA5: J7.8 (Pin_8), U2.7 (PA5)
- new net 2PA6: J7.9 (Pin_9), U2.8 (PA6)
- new net 2PA7: J7.10 (Pin_10), U2.9 (PA7)
- new net 2PB0: J8.3 (Pin_3), U2.10 (PB0)
- new net 2PB1: J8.4 (Pin_4), U2.11 (PB1)
- new net 2PB2: J8.5 (Pin_5), U2.12 (PB2)
- new net 2PB3: J8.6 (Pin_6), U2.13 (PB3)
- new net 2PB4: J8.7 (Pin_7), U2.14 (PB4)
- new net 2PB5: J8.8 (Pin_8), U2.15 (PB5)
- new net 2PB6: J8.9 (Pin_9), U2.16 (PB6)
- new net 2PB7: J8.10 (Pin_10), U2.17 (PB7)
- new net ~{CS_V2}: J6.1 (Pin_1), J6.3 (Pin_3), J6.5 (Pin_5), J6.7 (Pin_7), U2.23 (~{CS2})
- new net ~{IRQ_V2}: D3.1 (K), U2.21 (~{IRQ})
Other:
- moved on the sheet: D2

Commit message: Routing PCB
Parts:
- removed J5: IO VIA1, Connector_PinHeader_2.54mm:PinHeader_2x04_P2.54mm_Vertical, symbol Connector_Generic:Conn_02x04_Odd_Even
- removed J6: IO VIA2, Connector_PinHeader_2.54mm:PinHeader_2x04_P2.54mm_Vertical, symbol Connector_Generic:Conn_02x04_Odd_Even
- added C1, C2: .1uF, Capacitor_THT:C_Disc_D4.3mm_W1.9mm_P5.00mm, symbol Device:C
- added J9: VIA IO Select, Connector_PinHeader_2.54mm:PinHeader_3x06_P2.54mm_Vertical, symbol Connector_Generic:Conn_03x06_AB_Select_Letter_Last
- renumbered C1 to C3
Connections:
- net CA1: no longer J4.11 (Pin_11)
- net CB1: now also J4.11 (Pin_11)
- net GND: now also C1.2, C2.2
- net VCC: now also C1.1, C2.1
- net ~{CS_V1}: now also J9.1a (Pin_1a), J9.2a (Pin_2a), J9.3a (Pin_3a), J9.4a (Pin_4a), J9.5a (Pin_5a), J9.6a (Pin_6a)
- net ~{CS_V2}: now also J9.1b (Pin_1b), J9.2b (Pin_2b), J9.3b (Pin_3b), J9.4b (Pin_4b), J9.5b (Pin_5b), J9.6b (Pin_6b)
- net ~{IO_03}: now also J9.2 (Pin_2)
- net ~{IO_04}: now also J9.3 (Pin_3)
- net ~{IO_05}: now also J9.4 (Pin_4)
- net ~{IO_06}: now also J9.5 (Pin_5)
- net ~{IO_07}: now also J9.6 (Pin_6)
- net ~{IO_SLOT}: now also J9.1 (Pin_1)
Other:
- moved on the sheet: D2, D3, J3, J4, J7, J8, R3, U1

Commit message: IOCard with SMD bypass caps
Parts:
- C1, C2: footprint Capacitor_THT:C_Disc_D4.3mm_W1.9mm_P5.00mm -> Capacitor_SMD:C_1206_3216Metric_Pad1.33x1.80mm_HandSolder
Changed lines of the file:
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@@
       (effects (font (size 1.27 1.27)) (justify left))
     )
-    (property "Footprint" "Capacitor_THT:C_Disc_D4.3mm_W1.9mm_P5.00mm" (at 246.0752 33.02 0)
+    (property "Footprint" "Capacitor_SMD:C_1206_3216Metric_Pad1.33x1.80mm_HandSolder" (at 246.0752 33.02 0)
       (effects (font (size 1.27 1.27)) hide)
     )
@@
       (effects (font (size 1.27 1.27)) (justify left))
     )
-    (property "Footprint" "Capacitor_THT:C_Disc_D4.3mm_W1.9mm_P5.00mm" (at 257.5052 33.02 0)
-      (effects (font (size 1.27 1.27)) hide)
-    )
+    (property "Footprint" "Capacitor_SMD:C_1206_3216Metric_Pad1.33x1.80mm_HandSolder" (at 257.5052 33.02 0)
+      (effects (font (size 1.27 1.27)) hide)
+    )
